Commit message: added hardware control. but at this point one of the servos got damaged

File: buddy_arm_description/urdf/buddy_core.urdf.xacro (robot description, xacro)
@@ -16,16 +16,4 @@
   <xacro:property name="base_height" value="0.055"/>
   <xacro:property name="PI" value="3.142593"/>
-  <material name="blue">
-      <color rgba="0.0 0.0 1.0 1.0"/>
-  </material>
-  <material name="red">
-      <color rgba="1.0 0.0 0.0 1.0"/>
-  </material>
-  <material name="green">
-      <color rgba="0.0 1.0 0.0 1.0"/>
-  </material>
-  <material name="yellow">
-      <color rgba="1.0 1.0 0.0 1.0"/>
-  </material>
   <material name="white">
       <color rgba="1.0 1.0 1.0 1.0"/>
@@ -61,5 +49,5 @@
         <material name="white"/>
       </collision>
-      <xacro:box mass="50" length="${base_length}" width="${base_width}" height="${base_height}"
+      <xacro:box mass="1.0" length="${base_length}" width="${base_width}" height="${base_height}"
             xyz="0.0 0.0 ${-base_height/2}" rpy="0.0 0.0 0.0"/>
     </link>
@@ -225,12 +213,12 @@
       </visual>
       <collision>
-        <origin xyz="0.0 0.0 0.0" rpy="0.0 0.0 0.0"/>
-        <geometry>
-          <cylinder radius="${servo_radius}" length="${servo_length}"/>
-        </geometry>
-        <material name="black"/>
-      </collision>
-      <xacro:cylinder mass="0.069" radius="${servo_radius}" height="${servo_length}"
-            xyz="0.0 0.0 0.0" rpy="0.0 0.0 0.0"/>
+        <origin xyz="0.0 0.0 ${-servo_length/2}" rpy="0.0 0.0 0.0"/>
+        <geometry>
+          <cylinder radius="${servo_radius}" length="${servo_length}"/>
+        </geometry>
+        <material name="black"/>
+      </collision>
+      <xacro:cylinder mass="0.069" radius="${servo_radius}" height="${servo_length}"
+            xyz="0.0 0.0 ${-servo_length/2}" rpy="0.0 0.0 0.0"/>
     </link>
     <joint name="joint_5" type="revolute">
@@ -250,5 +238,5 @@
       </visual>
       <collision>
-        <origin xyz="0.0 0.0 0.0" rpy="0.0 0.0 0.0"/>
+        <origin xyz="${-gs_length/2} 0.0 0.0" rpy="0.0 0.0 0.0"/>
         <geometry>
           <box size="${gs_length} ${gs_width} ${gs_height}"/>
@@ -257,5 +245,5 @@
       </collision>
       <xacro:box mass="0.05" length="${gs_length}" width="${gs_width}" height="${gs_height}"
-            xyz="0.0 0.0 0.0" rpy="0.0 0.0 0.0"/>
+           xyz="${-gs_length/2} 0.0 0.0" rpy="0.0 0.0 0.0"/>
     </link>
     <joint name="dummy3" type="fixed">
@@ -264,4 +252,28 @@
       <origin xyz="${gs_length} 0.0 ${-servo_length/2}" rpy="0.0 0.0 0.0"/>
     </joint>
+    <link name="gripper_right">
+      <visual>
+          <origin rpy="0 0 0" xyz="-0.06 0.0 0.0"/>
+          <geometry>
+              <mesh filename="package://buddy_arm_description/meshes/left_finger.STL" scale="0.001 0.001 0.001"/>
+          </geometry>
+      </visual>
+      <collision>
+        <origin rpy="0 0 0" xyz="-0.06 0.0 0.0"/>
+          <geometry>
+              <mesh filename="package://buddy_arm_description/meshes/left_finger.STL" scale="0.001 0.001 0.001"/>
+          </geometry>
+      </collision>
+      <xacro:box mass="0.05" length="${gs_length}" width="${gs_width}" height="${gs_height}"
+            rpy="0 0 0" xyz="-0.06 0.0 0.0"/>
+  </link>
+  <joint name ="joint_6" type="revolute">
+    <parent link="gripper_support"/>
+    <child link = "gripper_right"/>
+    <origin xyz="0.0 0.0 ${-gs_height/2}" rpy="${PI/2} 0.0 ${PI}"/>
+    <axis xyz="0 0 1"/>
+    <limit lower="0.0" upper="${PI/2}"
+           effort="1000" velocity="10"/>
+  </joint>
     <link name="gripper_left">
       <visual>
@@ -278,7 +290,7 @@
       </collision>
       <xacro:box mass="0.05" length="${gs_length}" width="${gs_width}" height="${gs_height}"
-            xyz="0.0 0.0 0.0" rpy="0.0 0.0 0.0"/>
+          rpy="0 0 0" xyz="-0.06 ${-gs_height/2} 0.0"/>
   </link>
-  <joint name ="joint_6" type="revolute">
+  <joint name ="joint_7" type="revolute">
     <parent link="gripper_support"/>
     <child link = "gripper_left"/>
@@ -287,29 +299,12 @@
     <limit lower="${-PI / 2}" upper="0.0"
            effort="1000" velocity="10"/>
+           <mimic joint="joint_6" multiplier="-1"/>
   </joint>
-  <link name="gripper_right">
-    <visual>
-        <origin rpy="0 0 0" xyz="-0.06 0.0 0.0"/>
-        <geometry>
-            <mesh filename="package://buddy_arm_description/meshes/left_finger.STL" scale="0.001 0.001 0.001"/>
-        </geometry>
-    </visual>
-    <collision>
-      <origin rpy="0 0 0" xyz="-0.06 0.0 0.0"/>
-        <geometry>
-            <mesh filename="package://buddy_arm_description/meshes/left_finger.STL" scale="0.001 0.001 0.001"/>
-        </geometry>
-    </collision>
-    <xacro:box mass="0.05" length="${gs_length}" width="${gs_width}" height="${gs_height}"
-            xyz="0.0 0.0 0.0" rpy="0.0 0.0 0.0"/>
-</link>
-<joint name ="joint_7" type="revolute">
-  <parent link="gripper_support"/>
-  <child link = "gripper_right"/>
-  <origin xyz="0.0 0.0 ${-gs_height/2}" rpy="${PI/2} 0.0 ${PI}"/>
-  <axis xyz="0 0 1"/>
-  <limit lower="0.0" upper="${PI/2}"
-         effort="1000" velocity="10"/>
-</joint>
+  <!-- my fix for moveit -->
+  <joint name="joint_7_mimic" type="fixed">
+    <parent link="world" />
+    <child link="random" />
+  </joint>
+  <link name="random"/>
     <xacro:arm_default_transmission joint_number="1"></xacro:arm_default_transmission>
     <xacro:arm_default_transmission joint_number="2"></xacro:arm_default_transmission>

File: buddy_arm_description/urdf/buddy_gazebo.urdf.xacro (robot description, xacro)
@@ -7,9 +7,6 @@
         <material>Gazebo/White</material>
     </gazebo>
-    <gazebo reference="link7">
+    <gazebo reference="gripper_support">
         <material>Gazebo/White</material>
-    </gazebo>
-    <gazebo reference="tool_tip">
-        <material>Gazebo/Yellow</material>
     </gazebo>
     <gazebo reference="link1">
@@ -28,5 +25,5 @@
         <material>Gazebo/Black</material>
     </gazebo>
-    <gazebo reference="link8">
+    <gazebo reference="link7">
         <material>Gazebo/Black</material>
     </gazebo>
@@ -35,5 +32,5 @@
           <robot_param>robot_description</robot_param>
           <robot_param_node>robot_state_publisher</robot_param_node>
-          <!-- <parameters>$(find arm_controller)/config/robotarm_controllers.yaml</parameters> -->
+          <parameters>$(find buddy_arm_controller)/config/buddy_arm_controllers.yaml</parameters>
         </plugin>
       </gazebo>

File: buddy_arm_description/urdf/buddy_ros2_control.urdf.xacro (robot description, xacro)
@@ -1,4 +1,4 @@
 <?xml version="1.0"?>
-<robot xmlns:xacro="http://www.ros.org/wiki/xacro">
+<robot xmlns:xacro="http://ros.org/wiki/xacro">
     <ros2_control name="RobotSystem" type="system">
         <xacro:if value="$(arg is_sim)">
@@ -6,4 +6,11 @@
                 <plugin>gazebo_ros2_control/GazeboSystem</plugin>
             </hardware>
+             <joint name="joint_7">
+            <param name="mimic">joint_6</param>
+            <param name="multiplier">-1</param>
+            <command_interface name="position"/>
+            <state_interface name="position"/>
+            <limit lower="${-PI/2}" upper="0" effort="1000" velocity="10"/>
+        </joint>
         </xacro:if>
         <xacro:unless value="$(arg is_sim)">
@@ -14,44 +21,32 @@
         </xacro:unless>
         <joint name="joint_1">
-            <command_interface name="position">
-            <param name="min">0</param>
-            <param name="max">3.142</param>
-            </command_interface>
+            <command_interface name="position"/>
             <state_interface name="position"/>
+            <limit lower="0" upper="${PI}" effort="1000" velocity="10"/>
         </joint>
         <joint name="joint_2">
-            <command_interface name="position">
-            <param name="min">0</param>
-            <param name="max">3.142</param>
-            </command_interface>
+            <command_interface name="position"/>
             <state_interface name="position"/>
+            <limit lower="0" upper="${PI}" effort="1000" velocity="10"/>
         </joint>
         <joint name="joint_3">
-            <command_interface name="position">
-            <param name="min">0</param>
-            <param name="max">3.142</param>
-            </command_interface>
+            <command_interface name="position"/>
             <state_interface name="position"/>
+            <limit lower="0" upper="${PI}" effort="1000" velocity="10"/>
         </joint>
         <joint name="joint_4">
-            <command_interface name="position">
-            <param name="min">0</param>
-            <param name="max">3.142</param>
-            </command_interface>
+            <command_interface name="position"/>
             <state_interface name="position"/>
+            <limit lower="0" upper="${PI}" effort="1000" velocity="10"/>
         </joint>
         <joint name="joint_5">
-            <command_interface name="position">
-            <param name="min">0</param>
-            <param name="max">3.142</param>
-            </command_interface>
+            <command_interface name="position"/>
             <state_interface name="position"/>
+            <limit lower="0" upper="${PI}" effort="1000" velocity="10"/>
         </joint>
         <joint name="joint_6">
-            <command_interface name="position">
-            <param name="min">0</param>
-            <param name="max">3.142</param>
-            </command_interface>
+            <command_interface name="position"/>
             <state_interface name="position"/>
+            <limit lower="0" upper="${PI/2}" effort="1000" velocity="10"/>
         </joint>
     </ros2_control>
