Commit message: fixed simulation

File: src/buddy_arm_description/urdf/buddy_gazebo.urdf.xacro (robot description, xacro)
@@ -25,7 +25,7 @@
         <material>Gazebo/Black</material>
     </gazebo>
-    <gazebo reference="link7">
+    <!-- <gazebo reference="link7">
         <material>Gazebo/Black</material>
-    </gazebo>
+    </gazebo> -->
     <gazebo>
         <plugin filename="libgazebo_ros2_control.so" name="buddy_ros2_control">

File: src/buddy_arm_description/urdf/buddy_ros2_control.urdf.xacro (robot description, xacro)
@@ -6,6 +6,6 @@
                 <plugin>gazebo_ros2_control/GazeboSystem</plugin>
             </hardware>
-             <joint name="joint_7">
-            <param name="mimic">joint_6</param>
+             <joint name="joint_6">
+            <param name="mimic">joint_5</param>
             <param name="multiplier">-1</param>
             <command_interface name="position"/>
@@ -43,9 +43,4 @@
             <command_interface name="position"/>
             <state_interface name="position"/>
-            <limit lower="0" upper="${PI}" effort="1000" velocity="10"/>
-        </joint>
-        <joint name="joint_6">
-            <command_interface name="position"/>
-            <state_interface name="position"/>
             <limit lower="0" upper="${PI/2}" effort="1000" velocity="10"/>
         </joint>
