Commit message: simulation working now

File: src/buddy_arm_description/urdf/buddy_core.urdf.xacro (robot description, xacro)
@@ -273,5 +273,5 @@
     <origin xyz="0.0 0.0 ${-gs_height/2}" rpy="${PI/2} 0.0 ${PI}"/>
     <axis xyz="0 0 1"/>
-    <limit lower="0.0" upper="${PI/2}"
+    <limit lower="0.0" upper="${PI/4}"
            effort="1000" velocity="10"/>
   </joint>
@@ -297,5 +297,5 @@
     <origin xyz="0.0 0.0 ${gs_height/2}" rpy="${PI/2} 0.0 ${PI}"/>
     <axis xyz="0 0 1"/>
-    <limit lower="${-PI / 2}" upper="0.0"
+    <limit lower="${-PI/4}" upper="0.0"
            effort="1000" velocity="10"/>
            <mimic joint="joint_5" multiplier="-1"/>

File: src/buddy_arm_description/urdf/buddy_ros2_control.urdf.xacro (robot description, xacro)
@@ -11,5 +11,5 @@
             <command_interface name="position"/>
             <state_interface name="position"/>
-            <limit lower="${-PI/2}" upper="0" effort="1000" velocity="10"/>
+            <limit lower="${-PI/4}" upper="0" effort="1000" velocity="10"/>
         </joint>
         </xacro:if>
@@ -43,5 +43,5 @@
             <command_interface name="position"/>
             <state_interface name="position"/>
-            <limit lower="0" upper="${PI/2}" effort="1000" velocity="10"/>
+            <limit lower="0" upper="${PI/4}" effort="1000" velocity="10"/>
         </joint>
     </ros2_control>

Commit message: hardware

File: src/buddy_arm_description/urdf/buddy_core.urdf.xacro (robot description, xacro)
@@ -273,5 +273,5 @@
     <origin xyz="0.0 0.0 ${-gs_height/2}" rpy="${PI/2} 0.0 ${PI}"/>
     <axis xyz="0 0 1"/>
-    <limit lower="0.0" upper="${PI/4}"
+    <limit lower="0.0" upper="${7*PI/36}"
            effort="1000" velocity="10"/>
   </joint>
@@ -297,5 +297,5 @@
     <origin xyz="0.0 0.0 ${gs_height/2}" rpy="${PI/2} 0.0 ${PI}"/>
     <axis xyz="0 0 1"/>
-    <limit lower="${-PI/4}" upper="0.0"
+    <limit lower="${-7*PI/36}" upper="0.0"
            effort="1000" velocity="10"/>
            <mimic joint="joint_5" multiplier="-1"/>

File: src/buddy_arm_description/urdf/buddy_ros2_control.urdf.xacro (robot description, xacro)
@@ -11,5 +11,5 @@
             <command_interface name="position"/>
             <state_interface name="position"/>
-            <limit lower="${-PI/4}" upper="0" effort="1000" velocity="10"/>
+            <limit lower="${-7*PI/36}" upper="0" effort="1000" velocity="10"/>
         </joint>
         </xacro:if>
@@ -43,5 +43,5 @@
             <command_interface name="position"/>
             <state_interface name="position"/>
-            <limit lower="0" upper="${PI/4}" effort="1000" velocity="10"/>
+            <limit lower="0" upper="${7*PI/36}" effort="1000" velocity="10"/>
         </joint>
     </ros2_control>
